Commit message: r_control CPR calibration

File: description/robot_core.xacro (robot description, xacro)
@@ -71,5 +71,5 @@
         <collision>
             <geometry>
-                <cylinder radius="0.017" length="0.001" />
+                <cylinder radius="0.017" length="0.0001" />
             </geometry>
         </collision>

File: description/ros2_control.xacro (robot description, xacro)
@@ -11,5 +11,5 @@
                 <param name="baud_rate">57600</param>
                 <param name="timeout">1000</param>
-                <param name="enc_counts_per_rev">1601</param>
+                <param name="enc_counts_per_rev">482</param>  <!--1601-->
             </hardware>
             <joint name="left_wheel_joint">

Commit message: core restore and mapperyaml change

File: description/robot_core.xacro (robot description, xacro)
@@ -71,5 +71,5 @@
         <collision>
             <geometry>
-                <cylinder radius="0.017" length="0.0001" />
+                <cylinder radius="0.017" length="0.001" />
             </geometry>
         </collision>

Commit message: Controller&Core Descript Change

File: description/robot_core.xacro (robot description, xacro)
@@ -38,5 +38,5 @@
             <origin xyz="0.1175 0 0.04" rpy="0 0 0"/>
             <geometry>
-                <box size="0.235 0.15 0.08"/>
+                <box size="0.235 0.10 0.08"/>
             </geometry>
             <material name="white"/>
@@ -45,8 +45,8 @@
             <origin xyz="0.1175 0 0.04" rpy="0 0 0"/>
             <geometry>
-                <box size="0.235 0.15 0.08"/>
+                <box size="0.235 0.10 0.08"/>
             </geometry>
         </collision>
-        <xacro:inertial_box mass="0.5" x="0.235" y="0.15" z="0.08">
+        <xacro:inertial_box mass="0.5" x="0.235" y="0.10" z="0.08">
             <origin xyz="0.1175 0 0.04" rpy="0 0 0"/>
         </xacro:inertial_box>
@@ -59,5 +59,5 @@
         <parent link="base_link"/>
         <child link="left_wheel"/>
-        <origin xyz="-0.04 0.087 0" rpy="-${pi/2} 0 0"/>
+        <origin xyz="-0.04 0.055 0" rpy="-${pi/2} 0 0"/>
         <axis xyz="0 0 1"/>
     </joint>
@@ -65,5 +65,5 @@
         <visual>
             <geometry>
-                <cylinder radius="0.017" length="0.02" />
+                <cylinder radius="0.022" length="0.02" />
             </geometry>
             <material name="blue"/>
@@ -71,8 +71,8 @@
         <collision>
             <geometry>
-                <cylinder radius="0.017" length="0.001" />
+                <cylinder radius="0.022" length="0.001" />
             </geometry>
         </collision>
-        <xacro:inertial_cylinder mass="0.1" length="0.02" radius="0.017">
+        <xacro:inertial_cylinder mass="0.1" length="0.02" radius="0.022">
         <origin xyz="0 0 0" rpy="0 0 0"/>
     </xacro:inertial_cylinder>
@@ -85,5 +85,5 @@
         <parent link="base_link"/>
         <child link="right_wheel"/>
-        <origin xyz="-0.04 -0.087 0" rpy="${pi/2} 0 0"/>
+        <origin xyz="-0.04 -0.055 0" rpy="${pi/2} 0 0"/>
         <axis xyz="0 0 -1"/>
     </joint>
@@ -91,5 +91,5 @@
         <visual>
             <geometry>
-                <cylinder radius="0.017" length="0.02" />
+                <cylinder radius="0.022" length="0.02" />
             </geometry>
             <material name="blue"/>
@@ -97,8 +97,8 @@
         <collision>
             <geometry>
-                <cylinder radius="0.017" length="0.001" />
+                <cylinder radius="0.022" length="0.001" />
             </geometry>
         </collision>
-        <xacro:inertial_cylinder mass="0.1" length="0.02" radius="0.017">
+        <xacro:inertial_cylinder mass="0.1" length="0.02" radius="0.022">
         <origin xyz="0 0 0" rpy="0 0 0"/>
     </xacro:inertial_cylinder>
